Commit message: LET'S GOOOOOO SOOOO SOOOO SOOO MCUH CODING OMG

File: src/uav_gimbal/robot_description/uavGimbal.urdf (robot description, URDF)
Before this commit: robot robot, 9 links, 8 joints
Links:
- added link x_axis_cube, mass 0.01; collision box size=0.2 0.05 0.05; visual box size=2.5 0.05 0.05
- added link y_axis_cube, mass 0.01; collision box size=0.05 0.2 0.05; visual box size=0.05 2.5 0.05
- added link z_axis_cube, mass 0.01; collision box size=0.05 0.05 0.2; visual box size=0.05 0.05 2.5
- link base_link: geometry collision box size=1 1 1; visual box size=0.1 0.1 0.1
Joints:
- added joint x_axis_joint: type fixed, parent uav_pitching, child x_axis_cube, origin xyz=0.15 0 0 rpy=0 0 0
- added joint y_axis_joint: type fixed, parent uav_pitching, child y_axis_cube, origin xyz=0 0.15 0 rpy=0 0 0
- added joint z_axis_joint: type fixed, parent uav_pitching, child z_axis_cube, origin xyz=0 0 0.15 rpy=0 0 0
- joint uav_pitching_to_cylinder0: limit lower=-3.14 upper=3.14 effort=1000.0 velocity=0.5 -> (none); type revolute -> continuous
